File: business_card.kicad_pcb (KiCad board)
At the start: 2 copper layers, 88.9 x 50.8 mm, 21 parts, among them J1 Conn_01x04_Pin, U1 STM32F042F4Px, U2 MIC5504-1.2YM5

Commit message: Added BOM and readme.
Parts:
- added G***: LOGO, LOGO, F.Cu at (81.0, 39.0)
- added G***: LOGO, LOGO, B.Cu at (122.6, 36.8)
Other:
- board text added: "1. Insert into USB 2. Open virtual COM port 3. _/('_')\_"
- board text added: "Daniel Adamkovic (947)-999-9999 private.email@pm.me"
- board text added: "Lorem ipsum dolor sit amet, consectetur adipiscing elit, sed do eiusmod tempor incididunt ut labore et dolore magna aliqua. Ut enim ad minim veniam, quis nostrud exercitation ullamco laboris nisi ut aliquip ex ea commodo consequat. Duis aute irure dolor in reprehenderit in voluptate velit esse cillum dolore eu fugiat nulla pariatur."
- board text added: "Resume"
