File: business_card.kicad_sch (KiCad schematic)
At the start: 21 parts, among them J1 Conn_01x04_Pin, U1 STM32F042F4Px, U2 MIC5504-1.2YM5

Commit message: Added BOM and readme.
Parts:
- BZ1: Price (none) -> 2.11; Source (none) -> https://www.mouser.com/ProductDetail/AATC/APD-1109-LF?qs=uw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
- C1, C2: value C_Small -> 1u; Price (none) -> 0.065; Source (none) -> https://www.mouser.com/ProductDetail/Samsung-Electro-Mechan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
- R1, R2, R3, R4, R5: value R_Small -> 2k
- R6: value R_Small -> 700
- U1: Price (none) -> 3.2; Source (none) -> https://www.mouser.com/ProductDetail/STMicroelectronics/STM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
- U2: Price (none) -> 0.25; Source (none) -> https://www.mouser.com/ProductDetail/Microchip-Technology/M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
Other:
- company: (none) -> N/A
- title: (none) -> Business Card
- moved on the sheet: BZ1, C1, D1, D2, D3, D4, D5, J1, R1, R2, R3, R4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
