File: hardware/business_card.kicad_sch (KiCad schematic)
At the start: 21 parts, among them J1 Conn_01x04_Pin, U1 STM32F042F4Px, U2 MIC5504-1.2YM5

Commit message: Updated readme
Parts:
- U1: value STM32F042F4Px -> STM32F042F6Px
Changed lines of the file:
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@@
       (effects (font (size 1.27 1.27)) (justify left))
     )
-    (property "Value" "STM32F042F4Px" (at 108.6359 119.38 0)
+    (property "Value" "STM32F042F6Px" (at 108.6359 119.38 0)
       (effects (font (size 1.27 1.27)) (justify left))
     )
@@
       (effects (font (size 1.27 1.27)) (justify right) hide)
     )
-    (property "Datasheet" "https://www.st.com/resource/en/datasheet/stm32f042f4.pdf" (at 106.68 96.52 0)
+    (property "Datasheet" "https://www.st.com/resource/en/datasheet/stm32f042f6.pdf" (at 106.68 96.52 0)
       (effects (font (size 1.27 1.27)) hide)
     )
